File: motordriver.kicad_sch (KiCad schematic)
At the start: 8 parts, among them J1 power terminal, J2 Screw_Terminal_01x02, J3 Screw_Terminal_01x02, J4 control pins, U1 L7805, U2 L293D

Commit message: footprints added
Parts:
- D1: footprint (none) -> LED_THT:LED_D3.0mm
- J1: footprint (none) -> TerminalBlock:TerminalBlock_bornier-2_P5.08mm
- J2: value Screw_Terminal_01x02 -> motor A; footprint (none) -> TerminalBlock:TerminalBlock_bornier-2_P5.08mm
- J3: value Screw_Terminal_01x02 -> motor B; footprint (none) -> TerminalBlock:TerminalBlock_bornier-2_P5.08mm
- J4: footprint (none) -> TerminalBlock:TerminalBlock_bornier-4_P5.08mm
- R1: footprint (none) -> Resistor_THT:R_Axial_DIN0309_L9.0mm_D3.2mm_P15.24mm_Horizontal
- U1: footprint (none) -> Package_DIP:Vishay_HVM-DIP-3_W7.62mm
Changed lines of the file:
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@@
 			)
 		)
-		(property "Value" "Screw_Terminal_01x02"
+		(property "Value" "motor B"
 			(at 173.99 125.7299 0)
 			(effects
@@
 			)
 		)
-		(property "Footprint" ""
+		(property "Footprint" "TerminalBlock:TerminalBlock_bornier-2_P5.08mm"
 			(at 171.45 123.19 0)
 			(effects
@@
 			)
 		)
-		(property "Value" "Screw_Terminal_01x02"
+		(property "Value" "motor A"
 			(at 173.99 110.4899 0)
 			(effects
@@
 			)
 		)
-		(property "Footprint" ""
+		(property "Footprint" "TerminalBlock:TerminalBlock_bornier-2_P5.08mm"
 			(at 171.45 107.95 0)
 			(effects
@@
 			)
 		)
-		(property "Footprint" ""
+		(property "Footprint" "LED_THT:LED_D3.0mm"
 			(at 196.85 66.04 0)
 			(effects
@@
 			)
 		)
-		(property "Footprint" ""
+		(property "Footprint" "Resistor_THT:R_Axial_DIN0309_L9.0mm_D3.2mm_P15.24mm_Horizontal"
 			(at 168.91 67.818 90)
 			(effects
@@
 			)
 		)
-		(property "Footprint" ""
+		(property "Footprint" "Package_DIP:Vishay_HVM-DIP-3_W7.62mm"
 			(at 133.985 64.77 0)
 			(effects
@@
 			)
 		)
-		(property "Footprint" ""
+		(property "Footprint" "TerminalBlock:TerminalBlock_bornier-2_P5.08mm"
 			(at 83.82 69.85 0)
 			(effects
@@
 			)
 		)
-		(property "Footprint" ""
+		(property "Footprint" "TerminalBlock:TerminalBlock_bornier-4_P5.08mm"
 			(at 68.58 113.03 0)
 			(effects

Commit message: pcb designed
Parts:
- J1, J2, J3: footprint TerminalBlock:TerminalBlock_bornier-2_P5.08mm -> TerminalBlock_Phoenix:TerminalBlock_Phoenix_MKDS-1,5-2-5.08_1x02_P5.08mm_Horizontal
- J4: footprint TerminalBlock:TerminalBlock_bornier-4_P5.08mm -> Connector_PinHeader_1.00mm:PinHeader_1x04_P1.00mm_Vertical
Changed lines of the file:
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@@
 			)
 		)
-		(property "Footprint" "TerminalBlock:TerminalBlock_bornier-2_P5.08mm"
+		(property "Footprint" "TerminalBlock_Phoenix:TerminalBlock_Phoenix_MKDS-1,5-2-5.08_1x02_P5.08mm_Horizontal"
 			(at 171.45 123.19 0)
 			(effects
@@
 			)
 		)
-		(property "Footprint" "TerminalBlock:TerminalBlock_bornier-2_P5.08mm"
+		(property "Footprint" "TerminalBlock_Phoenix:TerminalBlock_Phoenix_MKDS-1,5-2-5.08_1x02_P5.08mm_Horizontal"
 			(at 171.45 107.95 0)
 			(effects
@@
 			)
 		)
-		(property "Footprint" "TerminalBlock:TerminalBlock_bornier-2_P5.08mm"
+		(property "Footprint" "TerminalBlock_Phoenix:TerminalBlock_Phoenix_MKDS-1,5-2-5.08_1x02_P5.08mm_Horizontal"
 			(at 83.82 69.85 0)
 			(effects
@@
 			)
 		)
-		(property "Footprint" "TerminalBlock:TerminalBlock_bornier-4_P5.08mm"
+		(property "Footprint" "Connector_PinHeader_1.00mm:PinHeader_1x04_P1.00mm_Vertical"
 			(at 68.58 113.03 0)
 			(effects
